File: Hardware/SparkX_EZ_ARTIC_R2.brd (EAGLE design)
At the start: 10.7 x 40.6 mm, 114 parts, among them J25 U.FL, K1 TLP3475R, Q2 5.8A/30V/35mΩ, U1 ADM4210-1, U2 1.8V/100mA, U3 ARTIC_R2, U4 RFPA0133, U5 AS179-92LF, U6 3.0V, U7 SST25VF020BUSON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

Commit message: Routed
Parts:
- FD1, FD2, FD3, FD4: value FIDUCIAL1X2 -> FIDUCIALUFIDUCIAL; device SparkFun-Aesthetics:FIDUCIAL-1X2 -> SparkFun-Aesthetics:FIDUCIAL-MICRO
- moved CS0 22.9 mm to (0.64, 35.6)
- moved 1V8 19.8 mm to (10.0, 20.3), flipped to the bottom
- moved FRAME1 12.7 mm to (45.7, -10.2)
- moved FRAME2 12.7 mm to (45.7, -10.2)
- moved LOGO1 12.7 mm to (19.1, 50.8)
- moved LOGO3 11.5 mm to (14.0, 25.4)
- moved SPARKX2 11.5 mm to (14.0, 8.89)
- moved U$26 10.2 mm to (14.7, 18.8)
- moved FD1 4.97 mm to (8.26, 37.5)
- moved FD2 4.97 mm to (8.26, 37.5)
- moved FD3 4.02 mm to (1.52, 3.81)
- moved FD4 4.02 mm to (1.52, 3.81)
- moved L15 2.41 mm to (8.64, 18.0)
- moved C40 1.40 mm to (6.73, 18.0)
- moved R4 0.51 mm to (0.84, 14.5)
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Routing:
- net 1.8V: track 0.00 -> 39.8 mm, vias 0 -> 1
- net GND: track 82.8 -> 103.7 mm, vias 65 -> 62
- net INT1: track 3.99 -> 19.3 mm
- net CS0: track 32.5 -> 41.3 mm, vias 2 -> 3
- net 3.3V: track 65.3 -> 72.4 mm, vias 8 -> 10
- net VDD: track 90.9 -> 88.7 mm
- net N$6: track 0.01 -> 1.04 mm
- net N$13: track 6.21 -> 5.64 mm
- net GPIO0: track 40.5 -> 40.7 mm, vias 3 -> 2
- net N$3: vias 3 -> 2
Other:
- board text added: "JLCPCB JLC7628 4-Layer 0.8mm Impedance Control 4-Layer Board 0.8mm Thickness 1oz Copper (Outer layers) ENIG Finish When running the panelizer, add a vertical gap of 0.2" to make the boards easier to separate"
- board text removed: "JLCPCB JLC7628 4-Layer 0.8mm Impedance Control 4-Layer Board 0.8mm Thickness 1oz Copper (Outer layers) ENIG Finish Castellated Holes When running the panelizer, add a vertical gap of 0.2" to allow the castellated holes to be routed out"

Commit message: Ready for review
Parts:
- removed FRAME2: FRAME-LEDGER, SparkFun-Aesthetics:CREATIVE_COMMONS
- removed SPARKX2: SPARKX-LOGO4, SparkX:SPARKX-MEDIUM
- removed U$26: (no value), output:ARTIC_R20
- added GPIO0: TEST-POINT3, SparkFun-Connectors:PAD.03X.03
- added LOGO2: OSHW-LOGOMINI, SparkFun-Aesthetics:OSHW-LOGO-MINI
- added U$4: SPARKX-LOGO3, SparkX:SPARKX-SMALL
- added U$5, U$6: (no value), output:EZ_ARTIC_R20
- added U$8: SPARKX-LOGO2, SparkX:SPARKX-TINY
- L11, L12, L5, L6, L7, L8: device New_Parts_Coils:0402_COILCRAFT -> SparkFun-Coils:0402_COILCRAFT
- LOGO3: value OSHW-LOGOS -> OSHW-LOGOMINI; device SparkFun-Aesthetics:OSHW-LOGO-S -> SparkFun-Aesthetics:OSHW-LOGO-MINI
- moved LOGO3 11.5 mm to (6.48, 34.2), turned to 0 degrees
- moved FD3 3.42 mm to (0.64, 0.51)
- moved FD4 3.42 mm to (0.64, 0.51)
- renumbered VREF1 to 3V0
Connections:
- net GPIO0: now also GPIO0.P$1
Routing:
- net GPIO0: track 40.7 -> 44.7 mm, vias 2 -> 3
- net GND: track 103.7 -> 104.1 mm, vias 62 -> 68

Commit message: Ready for review
Parts:
- moved FD2 3.10 mm to (10.0, 40.0)
- moved C2 0.89 mm to (0.76, 7.56)
- moved R11 0.83 mm to (0.76, 9.53)
- moved R9 0.19 mm to (8.64, 7.30)
Routing:
- net V_BATT: track 41.6 -> 41.1 mm
- net FLASH_VCC: track 8.05 -> 8.57 mm
- net GND: vias 68 -> 69

Commit message: Review updates. Adding production files
Parts:
- added U$1: (no value), output:#OUT#0
- added U$2: (no value), output:#IN#0
- moved LOGO3 1.27 mm to (6.48, 32.9)
Connections:
- net V_BATT renamed PROC_PWR_EN
- net 1.8V: now also 1V8.1; no longer 1V8.P$1
- net CS0: now also CS0.1; no longer CS0.P$1
- net FLSH_CEN: now also FLSH_CEN.1; no longer FLSH_CEN.P$1
- net FLSH_SCLK: now also FLSH_SCLK.1; no longer FLSH_SCLK.P$1
- net FLSH_SI: now also FLSH_SI.1; no longer FLSH_SI.P$1
- net FLSH_SO: now also FLSH_SO.1; no longer FLSH_SO.P$1
- net GPIO0: now also GPIO0.1; no longer GPIO0.P$1
- net VDD: now also VDD.1; no longer VDD.P$1
- net VREF1: now also 3V0.1; no longer 3V0.P$1
Changed lines of the file:
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@@
 <element name="U$6" library="output" package="EZ_ARTIC_R20" value="" x="5.334" y="24.4475" smashed="yes" rot="MR0"/>
 <element name="LOGO2" library="SparkFun-Aesthetics" package="OSHW-LOGO-MINI" value="OSHW-LOGOMINI" x="8.128" y="39.116" smashed="yes" rot="R90"/>
-<element name="LOGO3" library="SparkFun-Aesthetics" package="OSHW-LOGO-MINI" value="OSHW-LOGOMINI" x="6.477" y="34.163" smashed="yes" rot="MR0"/>
+<element name="LOGO3" library="SparkFun-Aesthetics" package="OSHW-LOGO-MINI" value="OSHW-LOGOMINI" x="6.477" y="32.893" smashed="yes" rot="MR0"/>
 <element name="U$4" library="SparkX" package="SPARKX-SMALL" value="SPARKX-LOGO3" x="5.334" y="26.0985" smashed="yes" rot="MR0"/>
 <element name="U$8" library="SparkX" package="SPARKX-TINY" value="SPARKX-LOGO2" x="9.652" y="24.511" smashed="yes" rot="R90"/>
+<element name="U$1" library="output" package="#OUT#0" value="" x="5.334" y="4.8895" smashed="yes"/>
+<element name="U$2" library="output" package="#IN#0" value="" x="5.334" y="35.7505" smashed="yes" rot="MR0"/>
 </elements>
 <signals>
@@
 <contactref element="C19" pad="1"/>
 <contactref element="L1" pad="2"/>
-<contactref element="VDD" pad="P$1"/>
+<contactref element="VDD" pad="1"/>
 <contactref element="U8" pad="8"/>
 <contactref element="C51" pad="1"/>
@@
 <contactref element="U7" pad="6"/>
 <via x="8.382" y="13.0175" extent="1-16" drill="0.2"/>
-<contactref element="FLSH_SCLK" pad="P$1"/>
+<contactref element="FLSH_SCLK" pad="1"/>
 <wire x1="6.676" y1="12.323" x2="6.676" y2="12.3275" width="0.1524" layer="16"/>
 <wire x1="8.382" y1="13.0175" x2="8.382" y2="13.208" width="0.1524" layer="1"/>
@@
 <via x="9.3345" y="13.97" extent="1-16" drill="0.2"/>
 <contactref element="U7" pad="5"/>
-<contactref element="FLSH_SI" pad="P$1"/>
+<contactref element="FLSH_SI" pad="1"/>
 <wire x1="8.607" y1="14.014" x2="9.2905" y2="14.014" width="0.254" layer="1"/>
 <wire x1="9.2905" y1="14.014" x2="9.3345" y2="13.97" width="0.254" layer="1"/>
@@
 <via x="9.3345" y="14.5415" extent="1-16" drill="0.2"/>
 <contactref element="U7" pad="2"/>
-<contactref element="FLSH_SO" pad="P$1"/>
+<contactref element="FLSH_SO" pad="1"/>
 <wire x1="10.033" y1="13.843" x2="10.033" y2="12.827" width="0.1524" layer="16"/>
 <wire x1="10.033" y1="12.827" x2="10.033" y2="10.16" width="0.1524" layer="16"/>
@@
 <via x="9.3345" y="15.113" extent="1-16" drill="0.2"/>
 <contactref element="U7" pad="1"/>
-<contactref element="FLSH_CEN" pad="P$1"/>
+<contactref element="FLSH_CEN" pad="1"/>
 <wire x1="9.3345" y1="15.113" x2="8.8265" y2="14.605" width="0.1524" layer="16"/>
 <wire x1="8.8265" y1="14.605" x2="8.8265" y2="13.76251875" width="0.1524" layer="16"/>
@@
 <contactref element="U2" pad="5"/>
 <contactref element="C4" pad="1"/>
-<contactref element="1V8" pad="P$1"/>
+<contactref element="1V8" pad="1"/>
 <wire x1="1.4605" y1="26.789" x2="0.8175" y2="26.789" width="0.3048" layer="1"/>
 <wire x1="0.8175" y1="26.789" x2="0.3683" y2="26.3398" width="0.3048" layer="1"/>
@@
 <contactref element="C21" pad="2"/>
 <contactref element="K1" pad="3"/>
-<contactref element="3V0" pad="P$1"/>
+<contactref element="3V0" pad="1"/>
 <contactref element="G16" pad="2"/>
 <wire x1="0.6223" y1="33.8455" x2="0.743" y2="33.9662" width="0.1524" layer="1"/>
@@
 <wire x1="2.957" y1="12.8291" x2="3.0861" y2="12.7" width="0.1524" layer="1"/>
 <via x="3.0861" y="12.7" extent="1-16" drill="0.2"/>
-<contactref element="CS0" pad="P$1"/>
+<contactref element="CS0" pad="1"/>
 <wire x1="6.084" y1="39.8945" x2="6.084" y2="38.57348125" width="0.1524" layer="16"/>
 <wire x1="6.55428125" y1="38.1032" x2="6.604" y2="38.1032" width="0.1524" layer="16"/>
@@
 <wire x1="1.4351" y1="13.75300625" x2="1.4351" y2="10.18255625" width="0.127" layer="15"/>
 <wire x1="1.4351" y1="10.18255625" x2="2.54" y2="9.07765625" width="0.127" layer="15"/>
-<contactref element="GPIO0" pad="P$1"/>
+<contactref element="GPIO0" pad="1"/>
 <wire x1="1.446221875" y1="3.795721875" x2="1.573221875" y2="3.922721875" width="0.1524" layer="16"/>
 <wire x1="1.446221875" y1="3.795721875" x2="0.649278125" y2="3.795721875" width="0.1524" layer="16"/>
@@
 <wire x1="0.6731" y1="14.17641875" x2="0.6731" y2="3.2639" width="0.127" layer="15"/>
 <wire x1="0.6731" y1="3.2639" x2="1.2065" y2="2.7305" width="0.127" layer="15"/>
-</signal>
-<signal name="V_BATT">
-<contactref element="IN" pad="1"/>
-<contactref element="OUT" pad="1"/>
-<wire x1="9.084" y1="0.7455" x2="9.084" y2="1.083" width="0.3048" layer="1"/>
-<wire x1="9.084" y1="1.083" x2="9.3345" y2="1.3335" width="0.3048" layer="1"/>
-<wire x1="9.3345" y1="1.3335" x2="9.3345" y2="3.683" width="0.3048" layer="1"/>
-<wire x1="9.3345" y1="3.683" x2="10.287" y2="4.6355" width="0.3048" layer="1"/>
-<via x="9.779" y="38.227" extent="1-16" drill="0.2"/>
-<via x="10.287" y="38.227" extent="1-16" drill="0.2"/>
-<wire x1="10.287" y1="38.227" x2="9.779" y2="38.227" width="0.3048" layer="1"/>
-<wire x1="9.084" y1="39.8945" x2="9.084" y2="39.6205" width="0.3048" layer="16"/>
-<wire x1="10.287" y1="38.227" x2="10.033" y2="38.227" width="0.3048" layer="16"/>
-<wire x1="10.033" y1="38.227" x2="9.779" y2="38.227" width="0.3048" layer="16"/>
-<wire x1="10.287" y1="4.6355" x2="10.287" y2="38.227" width="0.3048" layer="1"/>
-<wire x1="10.033" y1="38.6715" x2="10.033" y2="38.227" width="0.3048" layer="16"/>
-<wire x1="9.084" y1="39.6205" x2="10.033" y2="38.6715" width="0.3048" layer="16"/>
 </signal>
 <signal name="3.3V">
@@
 <wire x1="1.524" y1="32.9565" x2="1.6637" y2="33.0962" width="0.1524" layer="1"/>
 </signal>
+<signal name="PROC_PWR_EN">
+<contactref element="IN" pad="1"/>
+<contactref element="OUT" pad="1"/>
+<wire x1="9.084" y1="0.7455" x2="9.084" y2="1.083" width="0.3048" layer="1"/>
+<wire x1="9.084" y1="1.083" x2="9.3345" y2="1.3335" width="0.3048" layer="1"/>
+<wire x1="9.3345" y1="1.3335" x2="9.3345" y2="3.683" width="0.3048" layer="1"/>
+<wire x1="9.3345" y1="3.683" x2="10.287" y2="4.6355" width="0.3048" layer="1"/>
+<via x="9.779" y="38.227" extent="1-16" drill="0.2"/>
+<via x="10.287" y="38.227" extent="1-16" drill="0.2"/>
+<wire x1="10.287" y1="38.227" x2="9.779" y2="38.227" width="0.3048" layer="1"/>
+<wire x1="10.287" y1="38.227" x2="10.033" y2="38.227" width="0.3048" layer="16"/>
+<wire x1="10.033" y1="38.227" x2="9.779" y2="38.227" width="0.3048" layer="16"/>
+<wire x1="10.287" y1="4.6355" x2="10.287" y2="38.227" width="0.3048" layer="1"/>
+<wire x1="9.084" y1="39.8945" x2="9.084" y2="39.303" width="0.3048" layer="16"/>
+<wire x1="9.084" y1="39.303" x2="9.2075" y2="39.1795" width="0.3048" layer="16"/>
+<wire x1="9.2075" y1="39.1795" x2="9.779" y2="39.1795" width="0.3048" layer="16"/>
+<wire x1="9.779" y1="39.1795" x2="10.033" y2="38.9255" width="0.3048" layer="16"/>
+<wire x1="10.033" y1="38.9255" x2="10.033" y2="38.227" width="0.3048" layer="16"/>
+</signal>
 </signals>
