File: Hardware/SparkX_EZ_ARTIC_R2.brd (EAGLE design)
At the start: 10.7 x 40.6 mm, 119 parts, among them J25 U.FL, K1 TLP3475R, Q2 5.8A/30V/35mΩ, U1 ADM4210-1, U2 1.8V/100mA, U3 ARTIC_R2, U4 RFPA0133, U5 AS179-92LF, U6 3.0V, U7 SST25VF020BUSON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

Commit message: Update 16-way FPC Connector
Parts:
- IN, OUT: value FPC_16_0.5MM_BACKFLIP -> (none); device New_Parts_Connectors:FPC_16_DOUBLESIDED_BACKFLIP -> SparkFun-Connectors:FPC_16_0.5MM
Changed lines of the file:
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@@
 <layers>
 <layer number="1" name="Top" color="4" fill="1" visible="yes" active="yes"/>
-<layer number="2" name="Route2" color="63" fill="1" visible="no" active="yes"/>
-<layer number="15" name="Route15" color="23" fill="1" visible="no" active="yes"/>
+<layer number="2" name="Route2" color="63" fill="1" visible="yes" active="yes"/>
+<layer number="15" name="Route15" color="23" fill="1" visible="yes" active="yes"/>
 <layer number="16" name="Bottom" color="1" fill="1" visible="yes" active="yes"/>
 <layer number="17" name="Pads" color="2" fill="1" visible="yes" active="yes"/>
@@
 <layer number="23" name="tOrigins" color="15" fill="1" visible="yes" active="yes"/>
 <layer number="24" name="bOrigins" color="15" fill="1" visible="yes" active="yes"/>
-<layer number="25" name="tNames" color="57" fill="1" visible="no" active="yes"/>
-<layer number="26" name="bNames" color="57" fill="1" visible="no" active="yes"/>
-<layer number="27" name="tValues" color="7" fill="1" visible="no" active="yes"/>
-<layer number="28" name="bValues" color="7" fill="1" visible="no" active="yes"/>
-<layer number="29" name="tStop" color="7" fill="3" visible="no" active="yes"/>
-<layer number="30" name="bStop" color="7" fill="6" visible="no" active="yes"/>
-<layer number="31" name="tCream" color="7" fill="4" visible="no" active="yes"/>
-<layer number="32" name="bCream" color="7" fill="5" visible="no" active="yes"/>
-<layer number="33" name="tFinish" color="6" fill="3" visible="no" active="yes"/>
-<layer number="34" name="bFinish" color="6" fill="6" visible="no" active="yes"/>
-<layer number="35" name="tGlue" color="7" fill="4" visible="no" active="yes"/>
-<layer number="36" name="bGlue" color="7" fill="5" visible="no" active="yes"/>
-<layer number="37" name="tTest" color="7" fill="1" visible="no" active="yes"/>
-<layer number="38" name="bTest" color="7" fill="1" visible="no" active="yes"/>
-<layer number="39" name="tKeepout" color="4" fill="11" visible="no" active="yes"/>
-<layer number="40" name="bKeepout" color="1" fill="11" visible="no" active="yes"/>
-<layer number="41" name="tRestrict" color="4" fill="10" visible="no" active="yes"/>
-<layer number="42" name="bRestrict" color="1" fill="10" visible="no" active="yes"/>
-<layer number="43" name="vRestrict" color="2" fill="10" visible="no" active="yes"/>
-<layer number="44" name="Drills" color="7" fill="1" visible="no" active="yes"/>
+<layer number="25" name="tNames" color="57" fill="1" visible="yes" active="yes"/>
+<layer number="26" name="bNames" color="57" fill="1" visible="yes" active="yes"/>
+<layer number="27" name="tValues" color="7" fill="1" visible="yes" active="yes"/>
+<layer number="28" name="bValues" color="7" fill="1" visible="yes" active="yes"/>
+<layer number="29" name="tStop" color="7" fill="3" visible="yes" active="yes"/>
+<layer number="30" name="bStop" color="7" fill="6" visible="yes" active="yes"/>
+<layer number="31" name="tCream" color="7" fill="4" visible="yes" active="yes"/>
+<layer number="32" name="bCream" color="7" fill="5" visible="yes" active="yes"/>
+<layer number="33" name="tFinish" color="6" fill="3" visible="yes" active="yes"/>
+<layer number="34" name="bFinish" color="6" fill="6" visible="yes" active="yes"/>
+<layer number="35" name="tGlue" color="7" fill="4" visible="yes" active="yes"/>
+<layer number="36" name="bGlue" color="7" fill="5" visible="yes" active="yes"/>
+<layer number="37" name="tTest" color="7" fill="1" visible="yes" active="yes"/>
+<layer number="38" name="bTest" color="7" fill="1" visible="yes" active="yes"/>
+<layer number="39" name="tKeepout" color="4" fill="11" visible="yes" active="yes"/>
+<layer number="40" name="bKeepout" color="1" fill="11" visible="yes" active="yes"/>
+<layer number="41" name="tRestrict" color="4" fill="10" visible="yes" active="yes"/>
+<layer number="42" name="bRestrict" color="1" fill="10" visible="yes" active="yes"/>
+<layer number="43" name="vRestrict" color="2" fill="10" visible="yes" active="yes"/>
+<layer number="44" name="Drills" color="7" fill="1" visible="yes" active="yes"/>
 <layer number="45" name="Holes" color="7" fill="1" visible="yes" active="yes"/>
-<layer number="46" name="Milling" color="3" fill="1" visible="no" active="yes"/>
-<layer number="47" name="Measures" color="7" fill="1" visible="no" active="yes"/>
-<layer number="48" name="Document" color="7" fill="1" visible="no" active="yes"/>
-<layer number="49" name="Reference" color="7" fill="1" visible="no" active="yes"/>
-<layer number="50" name="dxf" color="7" fill="1" visible="no" active="yes"/>
+<layer number="46" name="Milling" color="3" fill="1" visible="yes" active="yes"/>
+<layer number="47" name="Measures" color="7" fill="1" visible="yes" active="yes"/>
+<layer number="48" name="Document" color="7" fill="1" visible="yes" active="yes"/>
+<layer number="49" name="Reference" color="7" fill="1" visible="yes" active="yes"/>
+<layer number="50" name="dxf" color="7" fill="1" visible="yes" active="yes"/>
 <layer number="51" name="tDocu" color="6" fill="1" visible="yes" active="yes"/>
-<layer number="52" name="bDocu" color="7" fill="1" visible="no" active="yes"/>
+<layer number="52" name="bDocu" color="7" fill="1" visible="yes" active="yes"/>
 <layer number="3" name="Route3" color="17" fill="1" visible="no" active="no"/>
 <layer number="4" name="Route4" color="18" fill="1" visible="no" active="no"/>
@@
 <attribute name="PROD_ID" value="CAP-14993" x="7.112" y="3.1115" size="1.778" layer="28" ratio="15" rot="MR0" display="off"/>
 </element>
-<element name="IN" library="New_Parts_Connectors" package="FPC_16_DOUBLESIDED_BACKFLIP" value="FPC_16_0.5MM_BACKFLIP" x="5.334" y="38.5445" smashed="yes" rot="MR0">
-<attribute name="ATOM_PART" value="FPC05016-42201" x="5.334" y="38.5445" size="1.778" layer="28" font="vector" ratio="15" rot="MR0" display="off"/>
-<attribute name="PROD_ID" value="" x="5.334" y="38.5445" size="1.778" layer="28" font="vector" ratio="15" rot="MR0" display="off"/>
-</element>
-<element name="OUT" library="New_Parts_Connectors" package="FPC_16_DOUBLESIDED_BACKFLIP" value="FPC_16_0.5MM_BACKFLIP" x="5.334" y="2.0955" smashed="yes" rot="R180">
-<attribute name="ATOM_PART" value="FPC05016-42201" x="5.334" y="2.0955" size="1.778" layer="27" font="vector" ratio="15" rot="R180" display="off"/>
-<attribute name="PROD_ID" value="" x="5.334" y="2.0955" size="1.778" layer="27" font="vector" ratio="15" rot="R180" display="off"/>
+<element name="IN" library="SparkFun-Connectors" package="FPC_16_0.5MM" value="" x="5.334" y="38.5445" smashed="yes" rot="MR0">
+<attribute name="PROD_ID" value="CONN-16066" x="5.334" y="38.5445" size="1.778" layer="28" font="vector" ratio="15" rot="MR0" display="off"/>
+</element>
+<element name="OUT" library="SparkFun-Connectors" package="FPC_16_0.5MM" value="" x="5.334" y="2.0955" smashed="yes" rot="R180">
+<attribute name="PROD_ID" value="CONN-16066" x="5.334" y="2.0955" size="1.778" layer="27" font="vector" ratio="15" rot="R180" display="off"/>
 </element>
 <element name="FLSH_CEN" library="SparkFun-Connectors" package="PAD.03X.03" value="TEST-POINT3" x="10.033" y="17.78" smashed="yes" rot="MR0"/>
@@
 <signal name="3.3V">
 <contactref element="IN" pad="2"/>
-<contactref element="OUT" pad="2"/>
 <contactref element="IN" pad="15"/>
 <contactref element="OUT" pad="15"/>
@@
 <wire x1="8.001" y1="9.0805" x2="7.239" y2="9.0805" width="0.4064" layer="16"/>
 <wire x1="7.239" y1="9.0805" x2="6.35" y2="9.0805" width="0.4064" layer="16"/>
-<wire x1="8.584" y1="0.7455" x2="8.584" y2="1.472" width="0.3048" layer="1"/>
-<wire x1="8.584" y1="1.472" x2="8.636" y2="1.524" width="0.3048" layer="1"/>
 <via x="8.636" y="1.524" extent="1-16" drill="0.2"/>
 <wire x1="8.636" y1="1.524" x2="8.771" y2="1.659" width="0.3048" layer="16"/>
@@
 <wire x1="8.636" y1="5.1435" x2="8.636" y2="6.4525" width="0.4064" layer="1"/>
 <wire x1="7.239" y1="7.6835" x2="7.239" y2="9.0805" width="0.4064" layer="16"/>
+<contactref element="OUT" pad="2"/>
+<wire x1="8.636" y1="1.524" x2="8.584" y2="1.472" width="0.3048" layer="1"/>
+<wire x1="8.584" y1="1.472" x2="8.584" y2="0.7455" width="0.3048" layer="1"/>
 </signal>
 <signal name="V_USB">
