File: Hardware/SparkX_EZ_ARTIC_R2.sch (EAGLE design)
At the start: 113 parts, among them J25 U.FL, K1 TLP3475R, Q2 5.8A/30V/35mΩ, U1 ADM4210-1, U2 1.8V/100mA, U3 ARTIC_R2, U4 RFPA0133, U5 AS179-92LF, U6 3.0V, U7 SST25VF020BUSON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

Commit message: Routed
Parts:
- FD1, FD2, FD3, FD4: value FIDUCIAL1X2 -> FIDUCIALUFIDUCIAL; device SparkFun-Aesthetics:FIDUCIAL1X2 -> SparkFun-Aesthetics:FIDUCIALUFIDUCIAL
Changed lines of the file:
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@@
 <part name="FRAME1" library="SparkFun-Aesthetics" deviceset="FRAME-LEDGER" device=""/>
 <part name="LOGO1" library="SparkFun-Aesthetics" deviceset="SPECIAL_INSTRUCTIONS" device="-ORDERING"/>
-<part name="FD1" library="SparkFun-Aesthetics" deviceset="FIDUCIAL" device="1X2"/>
-<part name="FD2" library="SparkFun-Aesthetics" deviceset="FIDUCIAL" device="1X2"/>
-<part name="FD3" library="SparkFun-Aesthetics" deviceset="FIDUCIAL" device="1X2"/>
-<part name="FD4" library="SparkFun-Aesthetics" deviceset="FIDUCIAL" device="1X2"/>
+<part name="FD1" library="SparkFun-Aesthetics" deviceset="FIDUCIAL" device="UFIDUCIAL" value="FIDUCIALUFIDUCIAL"/>
+<part name="FD2" library="SparkFun-Aesthetics" deviceset="FIDUCIAL" device="UFIDUCIAL" value="FIDUCIALUFIDUCIAL"/>
+<part name="FD3" library="SparkFun-Aesthetics" deviceset="FIDUCIAL" device="UFIDUCIAL" value="FIDUCIALUFIDUCIAL"/>
+<part name="FD4" library="SparkFun-Aesthetics" deviceset="FIDUCIAL" device="UFIDUCIAL" value="FIDUCIALUFIDUCIAL"/>
 <part name="U3" library="New_Parts_IC-Comms" deviceset="ARTIC_R2" device=""/>
 <part name="U4" library="New_Parts_IC-Comms" deviceset="RFPA0133" device=""/>

Commit message: Ready for review
Parts:
- removed FRAME2: FRAME-LEDGER, SparkFun-Aesthetics:FRAME-LEDGER
- removed SPARKX2: SPARKX-LOGO4, SparkX:SPARKX-LOGO4
- removed VREF1: TEST-POINT3, SparkFun-Connectors:TEST-POINT3
- added 3V0, GPIO0: TEST-POINT3, SparkFun-Connectors:TEST-POINT3
- added LOGO2: OSHW-LOGOMINI, SparkFun-Aesthetics:OSHW-LOGOMINI
- added U$4: SPARKX-LOGO3, SparkX:SPARKX-LOGO3
- added U$8: SPARKX-LOGO2, SparkX:SPARKX-LOGO2
- L11: device New_Parts_Coils:30NH-0402 -> SparkFun-Coils:30NH-0402
- L12: device New_Parts_Coils:51NH-0402 -> SparkFun-Coils:51NH-0402
- L5: device New_Parts_Coils:15NH-0402 -> SparkFun-Coils:15NH-0402
- L6: device New_Parts_Coils:27NH-0402 -> SparkFun-Coils:27NH-0402
- L7: device New_Parts_Coils:18NH-0402 -> SparkFun-Coils:18NH-0402
- L8: device New_Parts_Coils:12NH-0402 -> SparkFun-Coils:12NH-0402
- LOGO3: value OSHW-LOGOS -> OSHW-LOGOMINI; device SparkFun-Aesthetics:OSHW-LOGOS -> SparkFun-Aesthetics:OSHW-LOGOMINI
Connections:
- net GPIO0: now also GPIO0.1
- net VREF1: now also 3V0.1; no longer VREF1.1
Other:
- note added: "Bottom"
- note added: "EZ Connectors"
- note added: "Top"
- note removed: "Connectors"
- note removed: "Paul Clark"

Commit message: Review updates. Adding production files
Connections:
- net V_BATT renamed PROC_PWR_EN
Other:
- moved on the sheet: C50, C51, IN, K1, L1, OUT, U7, U8

Commit message: Update 16-way FPC Connector
Parts:
- IN, OUT: value FPC_16_0.5MM_BACKFLIP -> (none); device New_Parts_Connectors:FPC_16_0.5MM_BACKFLIP -> SparkFun-Connectors:CONN_16FPC_16_0.5MM
Changed lines of the file:
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@@
 <part name="C50" library="SparkFun-Capacitors" deviceset="0.1UF" device="-0402T-6.3V-10%-X7R" value="0.1uF"/>
 <part name="GND55" library="SparkFun-PowerSymbols" deviceset="GND" device=""/>
-<part name="IN" library="New_Parts_Connectors" deviceset="FPC_16_0.5MM" device="_BACKFLIP"/>
-<part name="OUT" library="New_Parts_Connectors" deviceset="FPC_16_0.5MM" device="_BACKFLIP"/>
+<part name="IN" library="SparkFun-Connectors" deviceset="CONN_16" device="FPC_16_0.5MM"/>
+<part name="OUT" library="SparkFun-Connectors" deviceset="CONN_16" device="FPC_16_0.5MM"/>
 <part name="SUPPLY21" library="SparkFun-PowerSymbols" deviceset="3.3V" device=""/>
 <part name="SUPPLY22" library="SparkFun-PowerSymbols" deviceset="3.3V" device=""/>
@@
 <instance part="U$4" gate="G$1" x="307.34" y="7.62" smashed="yes"/>
 <instance part="U$8" gate="G$1" x="307.34" y="7.62" smashed="yes"/>
-<instance part="IN" gate="G$1" x="15.24" y="33.02" smashed="yes">
-<attribute name="NAME" x="12.7" y="53.594" size="1.778" layer="95"/>
-<attribute name="VALUE" x="12.7" y="7.62" size="1.778" layer="96"/>
-</instance>
-<instance part="OUT" gate="G$1" x="73.66" y="33.02" smashed="yes" rot="MR0">
-<attribute name="NAME" x="76.2" y="53.594" size="1.778" layer="95" rot="MR0"/>
-<attribute name="VALUE" x="76.2" y="7.62" size="1.778" layer="96" rot="MR0"/>
+<instance part="IN" gate="G$1" x="12.7" y="30.48" smashed="yes" rot="MR180">
+<attribute name="NAME" x="12.7" y="9.906" size="1.778" layer="95" rot="MR180"/>
+<attribute name="VALUE" x="10.16" y="55.88" size="1.778" layer="96" rot="MR180"/>
+</instance>
+<instance part="OUT" gate="G$1" x="76.2" y="30.48" smashed="yes" rot="R180">
+<attribute name="NAME" x="76.2" y="9.906" size="1.778" layer="95" rot="R180"/>
+<attribute name="VALUE" x="78.74" y="55.88" size="1.778" layer="96" rot="R180"/>
 </instance>
 <instance part="SUPPLY21" gate="G$1" x="25.4" y="53.34" smashed="yes">
@@
 <segment>
 <pinref part="SUPPLY21" gate="G$1" pin="3.3V"/>
-<wire x1="25.4" y1="53.34" x2="25.4" y2="48.26" width="0.1524" layer="91"/>
 <pinref part="IN" gate="G$1" pin="2"/>
-<wire x1="25.4" y1="48.26" x2="22.86" y2="48.26" width="0.1524" layer="91"/>
 <pinref part="IN" gate="G$1" pin="15"/>
+<wire x1="22.86" y1="48.26" x2="25.4" y2="48.26" width="0.1524" layer="91"/>
+<wire x1="25.4" y1="48.26" x2="25.4" y2="53.34" width="0.1524" layer="91"/>
 <wire x1="22.86" y1="15.24" x2="25.4" y2="15.24" width="0.1524" layer="91"/>
 <wire x1="25.4" y1="15.24" x2="25.4" y2="48.26" width="0.1524" layer="91"/>
@@
 <segment>
 <pinref part="SUPPLY22" gate="G$1" pin="3.3V"/>
-<wire x1="63.5" y1="53.34" x2="63.5" y2="48.26" width="0.1524" layer="91"/>
+<pinref part="OUT" gate="G$1" pin="15"/>
 <pinref part="OUT" gate="G$1" pin="2"/>
-<wire x1="63.5" y1="48.26" x2="66.04" y2="48.26" width="0.1524" layer="91"/>
-<pinref part="OUT" gate="G$1" pin="15"/>
+<wire x1="66.04" y1="48.26" x2="63.5" y2="48.26" width="0.1524" layer="91"/>
+<wire x1="63.5" y1="48.26" x2="63.5" y2="53.34" width="0.1524" layer="91"/>
 <wire x1="66.04" y1="15.24" x2="63.5" y2="15.24" width="0.1524" layer="91"/>
 <wire x1="63.5" y1="15.24" x2="63.5" y2="48.26" width="0.1524" layer="91"/>
@@
 <pinref part="IN" gate="G$1" pin="16"/>
 <wire x1="22.86" y1="12.7" x2="25.4" y2="12.7" width="0.1524" layer="91"/>
-<wire x1="25.4" y1="10.16" x2="25.4" y2="12.7" width="0.1524" layer="91"/>
-</segment>
-<segment>
+<wire x1="25.4" y1="12.7" x2="25.4" y2="10.16" width="0.1524" layer="91"/>
+</segment>
+<segment>
